Commit message: refactor(pan_tilt): scope topics + rename camera_link to avoid main-robot clash
So pan_tilt can coexist with grasp_bringup / the main-robot stack
without TF or latched-topic collisions:

- state_publisher now publishes to /pan_tilt/joint_states (private)
  instead of the shared /joint_states aggregator.
- pan_tilt.launch.py remaps robot_state_publisher's /robot_description
  and /joint_states to the /pan_tilt/ namespace. /tf and /tf_static
  stay global so downstream consumers still see one merged TF tree.
- Standalone URDF renames the camera link `camera_link` →
  `head_camera_link` to dodge the xarm_description's
  `link_eef → camera_link` edge when both bringups run together.
- Integration tests (t1/t3/t4) updated to look up the new link name.

File: src/pan_tilt/urdf/pan_tilt.urdf.xacro (robot description, xacro)
@@ -1,8 +1,14 @@
 <?xml version="1.0"?>
 <robot xmlns:xacro="http://www.ros.org/wiki/xacro" name="pan_tilt">
+  <!--
+    Link names are scoped to the head camera so this URDF can coexist with the
+    main robot URDF loaded by mobile_bringup (xarm_description already defines
+    `camera_link` under `link_eef`). `base_link` stays shared by design - the
+    pan axis is expressed in the robot's base_link frame.
+  -->
   <link name="base_link"/>
   <link name="pan_link"/>
   <link name="tilt_link"/>
-  <link name="camera_link"/>
+  <link name="head_camera_link"/>
   <joint name="pan_joint" type="revolute">
     <parent link="base_link"/>
@@ -21,5 +27,5 @@
   <joint name="camera_mount_joint" type="fixed">
     <parent link="tilt_link"/>
-    <child link="camera_link"/>
+    <child link="head_camera_link"/>
     <origin xyz="-0.0724 -0.009 0.075" rpy="0.107098723 -0.004162789 3.062236662"/>
   </joint>

Commit message: fix(pan_tilt): apply calibration joint offsets at runtime + harden against backward-camera basin
Two related issues caused the seat-recommend pipeline to project vision points
below ground in the HRI arm-pointing test:

1. The URDF chain ignored theta_p_offset / theta_t_offset entirely. The
   calibration FK in pan_tilt_model uses R_z(-(pan + p_off)) and
   R_y(tilt + t_off), but pan_tilt_state_publisher published raw firmware
   angles to /joint_states and the URDF applied them through R_z(-pan_joint)
   / R_y(+tilt_joint) with no offset baked in anywhere — silently
   mis-representing the camera's pose by up to ~45° (the parked-tilt angle).
   apply_to_urdf only patched the static T_A and camera_mount_joint and never
   wrote the offsets to any consumer.

2. cmd_chain's two-basin warm-start (basin0 vs basinπ) used an unstable
   min(rot_rmse) tie-breaker. On near-tied data the basin choice oscillated
   across recalibrations; once basinπ won, apply_to_urdf wrote a t_b_rotvec
   with body-frame yaw ≈ ±π — geometrically valid but tripping every
   downstream consumer that assumed a forward-facing camera.

Fixes deployed across four defense layers:

- Layer 1 (optimize.fit_chain / fit_joint): bound t_b_rotvec[Z] to ±π/2
  unless allow_flipped_camera=True. Forward-facing cameras must stay in
  basin0; bounded scipy.optimize.least_squares prevents the solver from
  drifting into the +π yaw basin under a noisy warm start.
- Layer 2 (optimize.warm_start_t_b_rotation): emit a UserWarning when
  back-solved yaw exceeds ±π/4 (suppressed when caller seeded basinπ
  intentionally). Earliest signal that an upstream optical→body conversion
  was missed.
- Layer 3 (apply_to_urdf): refuse to patch URDFs whose camera_mount_joint
  yaw exceeds ±π/2; new CalibrationApplyError with operator-facing message
  naming --allow-flipped-camera as the explicit override.
- Layer 4 (test/test_calibration.py): regression coverage — 7 new tests for
  bounds, warm-start warnings, patcher refusal/override paths, and the
  basin-selector preference.

Path A — runtime offsets (pan_tilt_state_publisher):
  declare pan_offset_rad / tilt_offset_rad parameters (default 0.0); add
  them to firmware feedback before publishing /joint_states. Convention
  matches the calibration FK: pan_joint axis 0 0 -1 → R_z(-(firmware +
  p_off)); tilt_joint axis 0 1 0 → R_y(+(firmware + t_off)). No URDF or
  launch-file change needed; pan_tilt.launch.py already passes the YAML
  config to the state publisher.

Path C — basin0 preference (run_calibration._prefer_basin_zero):
  prefer basin0 unless basinπ wins by more than 1° rot RMSE. Eliminates
  cross-recalibration basin oscillation on near-noiseless data while
  keeping basinπ available for genuinely flipped hardware (Tinker 2026's
  current pan-servo mounting requires it; basin0 fits 18° worse).

apply_to_urdf and run_calibration both now print the runtime offsets to
copy into pan_tilt.yaml after every successful run. utils.py exposes
`body_yaw_from_rotvec` and `rotvec_to_xyz_euler` as a single canonical
conversion shared by patcher, solver, warm-start, and tests.

calibration/readme.md gains a "Forward-camera invariant", "Runtime joint
offsets", and "Tinker 2026 is in basin-π" section so the operator
workflow is documented end-to-end.

Tests: 23 → 28 passing in test_calibration.py. Existing 90°-mount fixture
still passes (sits inside the ±π/2 yaw bound). State-publisher tests use
isolated topic names so they don't pick up live driver traffic.

Deployed (pan_tilt.yaml + urdf/pan_tilt.urdf.xacro):
  pan_offset_rad:  3.144957  (basinπ)
  tilt_offset_rad: -1.873517
  camera_mount_joint rpy: 0.117424 -1.14551 3.02469
  attach_xyz: -0.30101 -0.00768387 1.35858

File: src/pan_tilt/urdf/pan_tilt.urdf.xacro (robot description, xacro)
@@ -14,5 +14,5 @@
     <parent link="base_link"/>
     <child link="pan_link"/>
-    <origin xyz="-0.275369 -0.013443 1.545923" rpy="0.019631607 0.033441848 0.052035773"/>
+    <origin xyz="-0.30101 -0.00768387 1.35858" rpy="0.019631607 0.033441848 0.052035773"/>
     <axis xyz="0 0 -1"/>
     <limit lower="-3.141592653589793" upper="3.141592653589793" effort="1.0" velocity="10.0"/>
@@ -28,5 +28,5 @@
     <parent link="tilt_link"/>
     <child link="head_camera_link"/>
-    <origin xyz="-0.0724 -0.009 0.075" rpy="0.107098723 -0.004162789 3.062236662"/>
+    <origin xyz="0.0660332 0.0322669 0.0128519" rpy="0.117424 -1.14551 3.02469"/>
   </joint>
 </robot>
